Commit message: firefly_y6 gripper: Tianyi 总装 URDF + meshes; no-cache /assets
gr100_{base_link,L1,L2}.STL + firefly_y6_gr100.urdf = new gripper (claws axis
0 0 -1, mimic -1). NoCacheStaticFiles on /assets so the browser always re-fetches
updated meshes instead of serving a stale cached gripper.

File: soda_server/public/firefly_y6_gr100/firefly_y6_gr100.urdf (robot description, URDF)
Before this commit: robot firefly_y6_gr100, 11 links, 10 joints
Links:
- link gripper_base_link: mass 0.47163661 -> 0.26211
- link gripper_left_link_1: mass 0.02806607 -> 0.02755
- link gripper_right_link_1: mass 0.02806607 -> 0.02755
Joints:
- joint gripper_base_joint: origin xyz=0 0 0 rpy=0 0 0 -> xyz=0 0 0 rpy=0 0 1.5707963
- joint gripper_left_joint_1: axis -1 0 0 -> 0 0 -1; origin xyz=0 -0.015 0.076799 rpy=0 0 0 -> xyz=-0.015 0.01475 0.07679888 rpy=0 1.57079633 -1.57079633
- joint gripper_right_joint_1: axis 1 0 0 -> 0 0 -1; limit lower=0.0 upper=0.9 effort=5 velocity=10 -> lower=-0.9 upper=0.0 effort=5 velocity=10; mimic joint=gripper_left_joint_1 multiplier=1.0 offset=0 -> joint=gripper_left_joint_1 multiplier=-1.0 offset=0; origin xyz=0 0.015 0.076799 rpy=0 0 0 -> xyz=0.015 0.01475 0.07679888 rpy=0 1.57079633 -1.57079633
